Commit message: corrected geometry on camera link

File: description/camera.xacro (robot description, xacro)
@@ -9,5 +9,5 @@
         <visual>
             <geometry>
-                <box size="0.10 0.023 0.020"/>
+                <box size="0.023 0.10 0.020"/>
             </geometry>
             <material name="red"/>
@@ -15,8 +15,8 @@
         <collision>
             <geometry>
-                <box size="0.10 0.023 0.020"/>
+                 <box size="0.023 0.10 0.020"/>
             </geometry>
         </collision>
-        <xacro:inertial_box mass="0.063" x="0.10" y="0.023" z="0.020">
+        <xacro:inertial_box mass="0.063" x="0.023" y="0.10" z="0.020">
             <origin xyz="0 0 0" rpy="0 0 0"/>
         </xacro:inertial_box>

Commit message: added gazebo camera

File: description/camera.xacro (robot description, xacro)
@@ -9,18 +9,10 @@
         <visual>
             <geometry>
-                <box size="0.023 0.10 0.020"/>
+                <box size="0.010 0.03 0.03"/>
             </geometry>
             <material name="red"/>
         </visual>
-        <collision>
-            <geometry>
-                 <box size="0.023 0.10 0.020"/>
-            </geometry>
-        </collision>
-        <xacro:inertial_box mass="0.063" x="0.023" y="0.10" z="0.020">
-            <origin xyz="0 0 0" rpy="0 0 0"/>
-        </xacro:inertial_box>
     </link>
-     <joint name="camera_optical_joint" type="fixed">
+    <joint name="camera_optical_joint" type="fixed">
         <parent link="camera_link"/>
         <child link="camera_link_optical"/>
