Commit message: ccreated robot core xacro

File: description/robot_core.xacro (robot description, xacro)
@@ -48,4 +48,91 @@
       <material name="white" />
    </visual>
+   <collision>
+      <origin xyz="${chassis_length/2} 0 ${chassis_height/2}" rpy="0.0 0.0 0.0"/>
+      <geometry>
+         <box size="${chassis_length} ${chassis_width} ${chassis_height}"/>
+      </geometry>
+      <material name="white" />
+   </collision>
+   <xacro:inertial_box mass="0.1" x="0.247" y="0.2" z="0.068">
+        <origin xyz="${chassis_length/2} 0 ${chassis_height/2}"  rpy="0.0 0.0 0.0"/>
+      </xacro:inertial_box >
+</link>
+<!-- LEFT WHEEL -->
+<joint name="left_wheel_joint" type="continuous">
+   <parent link="base_link"/>
+   <child link="left_wheel"/>
+   <axis xyz="0 0 1"/>
+   <origin xyz="0 ${wheel_offset_y} 0" rpy="${-pi/2} 0 0"/>
+</joint>
+<link name="left_wheel">
+   <visual>
+      <origin xyz="0.0 0.0 0.0" rpy="0.0 0.0 0.0"/>
+      <geometry>
+         <cylinder radius="${wheel_radius}" length="${wheel_thickness}"/>
+      </geometry>
+      <material name="blue" />
+   </visual>
+   <collision>
+      <origin xyz="0.0 0.0 0.0" rpy="0.0 0.0 0.0"/>
+      <geometry>
+         <cylinder radius="${wheel_radius}" length="${wheel_thickness}"/>
+      </geometry>
+      <material name="blue" />
+   </collision>
+   <xacro:inertial_cylinder mass="${wheel_mass}" radius="${wheel_radius}" length="${wheel_thickness}" >
+      <origin xyz="0.0 0.0 0.0" rpy="0.0 0.0 0.0"/>
+    </xacro:inertial_cylinder >
+</link>
+<!-- RIGHT WHEEL -->
+<joint name="right_wheel_joint" type="continuous">
+   <parent link="base_link"/>
+   <child link="right_wheel"/>
+   <axis xyz="0 0 -1"/>
+   <origin xyz="0 ${-wheel_offset_y} 0" rpy="${pi/2} 0 0"/>
+</joint>
+<link name="right_wheel">
+   <visual>
+      <origin xyz="0.0 0.0 0.0" rpy="0 0.0 0.0"/>
+      <geometry>
+         <cylinder radius="${wheel_radius}" length="${wheel_thickness}"/>
+      </geometry>
+      <material name="blue" />
+   </visual>
+   <collision>
+      <origin xyz="0.0 0.0 0.0" rpy="0 0.0 0.0"/>
+      <geometry>
+         <cylinder radius="${wheel_radius}" length="${wheel_thickness}"/>
+      </geometry>
+      <material name="blue" />
+   </collision>
+   <xacro:inertial_cylinder mass="${wheel_mass}" radius="${wheel_radius}" length="${wheel_thickness}" >
+      <origin xyz="0.0 0.0 0.0" rpy="0.0 0.0 0.0"/>
+    </xacro:inertial_cylinder >
+</link>
+<!-- caster wheel -->
+<joint name="caster_wheel-joint" type="fixed">
+   <parent link="chassis"/>
+   <child link="caster_wheel"/>
+   <origin xyz="${caster_wheel_offset_x} 0.0 ${caster_wheel_offset_z}" rpy="0.0 0.0 0.0"/>
+</joint>
+<link name="caster_wheel">
+<visual>
+   <origin xyz="0.0 0.0 0.0" rpy="0.0 0.0 0.0"/>
+   <geometry>
+      <sphere radius="${caster_wheel_radius}"/>
+   </geometry>
+   <material name="black" />
+</visual>
+<collision>
+   <origin xyz="0.0 0.0 0.0" rpy="0.0 0.0 0.0"/>
+   <geometry>
+      <sphere radius="${caster_wheel_radius}"/>
+   </geometry>
+   <material name="black" />
+</collision>
+ <xacro:inertial_sphere mass="${caster_wheel_mass}" radius="${caster_wheel_radius}">
+      <origin xyz="0.0 0.0 0.0" rpy="0.0 0.0 0.0"/>
+</xacro:inertial_sphere>
 </link>
 </robot>

Commit message: added simulation launch file

File: description/robot_core.xacro (robot description, xacro)
@@ -59,4 +59,7 @@
       </xacro:inertial_box >
 </link>
+ <gazebo reference="chassis">
+    <material>Gazebo/White</material>
+  </gazebo>
 <!-- LEFT WHEEL -->
 <joint name="left_wheel_joint" type="continuous">
@@ -85,4 +88,7 @@
     </xacro:inertial_cylinder >
 </link>
+ <gazebo reference="left_wheel">
+    <material>Gazebo/Blue</material>
+  </gazebo>
 <!-- RIGHT WHEEL -->
 <joint name="right_wheel_joint" type="continuous">
@@ -111,4 +117,7 @@
     </xacro:inertial_cylinder >
 </link>
+ <gazebo reference="right_wheel">
+    <material>Gazebo/Blue</material>
+  </gazebo>
 <!-- caster wheel -->
 <joint name="caster_wheel-joint" type="fixed">
@@ -136,3 +145,8 @@
 </xacro:inertial_sphere>
 </link>
+<gazebo reference="caster_wheel">
+    <material>Gazebo/Black</material>
+    <mu1  value="0.05"/>
+    <mu2  value="0.05"/>
+  </gazebo>
 </robot>
