Commit message: added launch file for depth camera

File: description/depth_camera.xacro (robot description, xacro)
@@ -16,5 +16,5 @@
     <joint name="camera_optical_joint" type="fixed">
         <parent link="camera_link"/>
-        <child link="camera_link_optical"/>
+        <child link="camera_depth_link_optical"/>
         <origin xyz="0 0 0" rpy="${-pi/2} 0 ${-pi/2}"/>
     </joint>
