Commit message: modified gazebo_control

File: description/gazebo_control.xacro (robot description, xacro)
@@ -1,33 +1,20 @@
 <?xml version="1.0"?>
-<robot xmlns:xacro="http://www.ros.org/wiki/xacro" name="robot">
+<robot xmlns:xacro="http://www.ros.org/wiki/xacro">
     <gazebo>
-        <plugin name='differential_drive_controller' filename='libgazebo_ros_diff_drive.so'>
-            <!-- Misc configs-->
-            <alwaysOn>true</alwaysOn>
-            <legacyMode>false</legacyMode>
-            <updateRate>10</updateRate>
-            <rosDebugLevel>na</rosDebugLevel>
+        <plugin name="diff_drive" filename="libgazebo_ros_diff_drive.so">
             <!-- Wheel Information -->
-            <wheelSeparation>0.225</wheelSeparation>
-            <wheelDiameter>0.0675</wheelDiameter>
-            <!-- Joints -->
-            <leftJoint>left_wheel_joint</leftJoint>
-            <rightJoint>right_wheel_joint</rightJoint>
+            <left_joint>left_wheel_joint</left_joint>
+            <right_joint>right_wheel_joint</right_joint>
+            <wheel_separation>0.225</wheel_separation>
+            <wheel_diameter>0.0675</wheel_diameter>
             <!-- Limits -->
-            <wheelTorque>10</wheelTorque>
-            <wheelAcceleration>2.0</wheelAcceleration>
-            <torque>5</torque>
-            <!-- topics  -->
-            <commandTopic>cmd_vel</commandTopic>
-            <odometryTopic>odom</odometryTopic>
-            <odometrySource>world</odometrySource>    <!-- odometrySource options "world" "encoder" -->
-            <!-- Frames -->
-            <odometryFrame>odom</odometryFrame>
-            <robotBaseFrame>base_link</robotBaseFrame>
-            <!-- outputs -->
-            <publishTf>1</publishTf>
-            <publishOdomTF>true</publishOdomTF>
-            <publishWheelTF>true</publishWheelTF>
-            <publishWheelJointState>true</publishWheelJointState>
+            <max_wheel_torque>200</max_wheel_torque>
+            <max_wheel_acceleration>10.0</max_wheel_acceleration>
+            <!-- Output -->
+            <odometry_frame>odom</odometry_frame>
+            <robot_base_frame>base_link</robot_base_frame>
+            <publish_odom>true</publish_odom>
+            <publish_odom_tf>true</publish_odom_tf>
+            <publish_wheel_tf>true</publish_wheel_tf>
         </plugin>
     </gazebo>

File: description/robot_core.xacro (robot description, xacro)
@@ -128,3 +128,8 @@
      </xacro:inertial_sphere>
   </link>
+   <gazebo reference="caster_wheel_link">
+    <material>Gazebo/Red</material>
+    <mu1 value="0.001" />
+    <mu2 value="0.001" />
+  </gazebo>
 </robot>
